File: Shield IO/Isolate IO v.1.sch (EAGLE design)
At the start: 0 parts

Commit message: add reference design pdf
Parts:
- added C1, C5: (no value), rcl:CPOL-EUE2.5-5
- added C2, C6: (no value), rcl:CPOL-EUE3.5-10
- added C3, C4, C7, C8: (no value), rcl:C-EU025-030X050
- added D1, D10, D11, D12, D13, D14, D15, D16, D17, D18, D19, D2, D20, D21, D22, D23, D24, D25, D26, D27, D28, D3, D4, D5, D6, D7, D8, D9: (no value), diode:ZENER-DIODEZD-2.5
- added IC1, IC3: REG1117, burr-brown:REG1117
- added IC2, IC4: LD117AV28, v-reg:LD117AV28
- added OK1, OK10, OK11, OK12, OK13, OK14, OK15, OK16, OK17, OK18, OK19, OK2, OK20, OK3, OK4, OK5, OK6, OK7, OK8, OK9: PC817, optocoupler:PC817
- added X1, X10, X11, X12, X13, X14, X15, X2, X3, X4, X5, X6, X7, X8, X9: (no value), con-ptr500:AK500/3
Connections:
- new net N$1: D3.C, OK7.A
- new net N$10: D6.C, OK5.A
- new net N$11: D7.C, OK6.A
- new net N$12: D8.C, OK8.A
- new net N$13: D9.C, OK9.A
- new net N$14: D10.C, OK10.A
- new net N$15: D11.C, OK17.A
- new net N$16: D12.C, OK11.A
- new net N$17: D13.C, OK12.A
- new net N$18: D14.C, OK13.A
- new net N$19: D15.C, OK14.A
- new net N$2: C2.+, C3.1, IC3.VOUT, IC4.OUT
- new net N$20: D16.C, OK15.A
- new net N$21: D17.C, OK16.A
- new net N$22: D18.C, OK18.A
- new net N$23: D19.C, OK19.A
- new net N$24: D20.C, OK20.A
- new net N$25: D21.C, D3.A
- new net N$26: D1.A, D22.C
- new net N$27: D2.A, D23.C
- new net N$28: D24.C, D4.A
- new net N$29: D25.C, D5.A
- new net N$3: D1.C, OK1.A
- new net N$30: D26.C, D6.A
- new net N$31: D27.C, D7.A
- new net N$32: D28.C, D8.A
- new net N$4: C1.-, C2.-, C3.2, C4.2, C5.-, C6.-, C7.2, C8.2, D21.A, D22.A, D23.A, D24.A, D25.A, D26.A, D27.A, D28.A, IC1.GND, IC2.ADJ, IC3.GND, IC4.ADJ
- new net N$5: C6.+, C7.1, IC1.VOUT, IC2.OUT
- new net N$6: C1.+, C4.1, C5.+, C8.1, IC1.VIN, IC2.IN, IC3.VIN, IC4.IN
- new net N$7: D2.C, OK2.A
- new net N$8: D4.C, OK3.A
- new net N$9: D5.C, OK4.A
